File: zudo-pd.kicad_sch (KiCad schematic)
At the start: 0 parts

Commit message: feat: add hierarchical schematics and symbol library setup
KiCad Schematic Structure:
- Create hierarchical schematic design with 4 sub-sheets
  - usb-pd-input.kicad_sch (USB-PD input stage)
  - dc-dc-conversion.kicad_sch (DC-DC converters)
  - linear-regulation.kicad_sch (Linear regulators + protection)
  - output.kicad_sch (Output connectors)
- Update root schematic (zudo-pd.kicad_sch) with sheet symbols
- Update project configuration (zudo-pd.kicad_pro)

Symbol Library:
- Create /symbols/ directory for project symbols
- Add symbols/zudo-pd.kicad_sym (53KB, 24 symbols)
  - USB-TYPE-C-009 (USB-C connector, C2927029)
  - CH224D_C3975094 (USB-PD controller, C3975094)
  - LM7812_SMD, LM7912_SMD (voltage regulators)
  - Plus passives, connectors, and protection components
- Add sym-lib-table (symbol library configuration)

Documentation:
- Rename kicad-footprint-generation.md → kicad-parts-download.md
- Rewrite guide to cover BOTH footprints and symbols
  - Add clear explanation of footprints vs symbols
  - Add download options (both, footprint only, symbol only)
  - Add complete workflow with USB-C and CH224D examples
  - Add symbol library setup instructions
  - Update project structure to include /symbols/ directory
- Add footprint library setup screenshot
  - doc/static/kicad/footprint-library-setup.png (2.1MB)
  - Shows configured zudo-pd footprint library with ${KIPRJMOD} path
- Update kicad-workflow.md with library setup screenshot
- Update navigation (sidebars.js, how-to/index.md)

Project Structure:
- Establish parallel structure for libraries:
  - /footprints/kicad/*.kicad_mod (physical PCB pads)
  - /symbols/zudo-pd.kicad_sym (schematic symbols)
- Both use ${KIPRJMOD} for portable paths

🤖 Generated with [Claude Code](https://claude.com/claude-code)

Co-Authored-By: Claude Sonnet 4.5 <noreply@anthropic.com>
Other:
- added sheet DC-DC Conversion (dc-dc-conversion.kicad_sch)
- added sheet Linear Regulation (linear-regulation.kicad_sch)
- added sheet Output (output.kicad_sch)
- added sheet USB-PD Input (usb-pd-input.kicad_sch)
