File: zudo-pd.kicad_sch (KiCad schematic)
At the start: 0 parts

Commit message: wip
Other:
- sheet USB-PD Input ports: added none; removed +5V IN
Changed lines of the file:
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@@
-	)
-	(junction
-		(at 152.4 38.1)
-		(diameter 0)
-		(color 0 0 0 0)
 	)
 	(junction
@@
 	(wire
 		(pts
-			(xy 29.21 30.48) (xy 29.21 20.32)
-		)
-		(stroke
-			(width 0)
-			(type default)
-		)
-	)
-	(wire
-		(pts
 			(xy 148.59 64.77) (xy 105.41 64.77)
 		)
@@
 	(wire
 		(pts
-			(xy 33.02 30.48) (xy 29.21 30.48)
-		)
-		(stroke
-			(width 0)
-			(type default)
-		)
-	)
-	(wire
-		(pts
 			(xy 156.21 48.26) (xy 148.59 48.26)
-		)
-		(stroke
-			(width 0)
-			(type default)
-		)
-	)
-	(wire
-		(pts
-			(xy 152.4 20.32) (xy 152.4 38.1)
-		)
-		(stroke
-			(width 0)
-			(type default)
-		)
-	)
-	(wire
-		(pts
-			(xy 29.21 20.32) (xy 152.4 20.32)
 		)
 		(stroke
@@
 			(effects
 				(font
-					(size 1.27 1.27)
-				)
-				(justify left)
-			)
-		)
-		(pin "+5V IN" input
-			(at 33.02 30.48 180)
-			(effects
-				(font
