File: usb-pd-input.kicad_sch (KiCad schematic)
At the start: 0 parts

Commit message: wip
Parts:
- added C1: 10uF, easyeda2kicad:C1206, symbol zudo-pd:HGC1206R5106K500NSPJ
- added C2: 100nF, easyeda2kicad:C0805, symbol zudo-pd:CC0805KRX7R9BB104
- added C30: 1uF, easyeda2kicad:C0603, symbol zudo-pd:CGA0603X5R105K160JT
- added J1: USB-C, easyeda2kicad:TYPE-C-SMD_TYPE-C-6P, symbol zudo-pd:USB-TYPE-C-009
- added R11: 56k, easyeda2kicad:R0603, symbol zudo-pd:RT0603BRD0756KL
- added R12, R13: 5.1k, easyeda2kicad:R0603, symbol zudo-pd:0603WAF5101T5E
- added UU1: CH224D, easyeda2kicad:QFN-20_L3.0-W3.0-P0.40-BL-EP1.7, symbol zudo-pd:CH224D_C3975094
Connections:
- net GND: now also C1.1, C2.1, C30.2, J1.A12 (GND), J1.B12 (GND), R11.2, R12.1, R13.1, UU1.14 (ISP), UU1.15 (ISN), UU1.21 (GND), UU1.6 (~{NMOS})
- net USB-PD-power OUT: now also C1.2, C2.2, J1.A9 (VBUS), J1.B9 (VBUS), UU1.2 (VBUS)
- new net: J1.A5 (CC1), R12.2, R13.2, UU1.10 (CC1)
- new net: J1.B5 (CC2), UU1.11 (CC2)
- new net: R11.1, UU1.1 (DRV), UU1.19 (CFG1)
- new net: C30.1, UU1.7 (VDD)
- new net: UU1.8 (DP), UU1.9 (DM)
