File: usb-pd-input.kicad_sch (KiCad schematic)
At the start: 8 parts, among them J1 USB-C

Commit message: feat: KiCad回路図の更新（DC-DC変換段とリニアレギュレーション）
DC-DC変換段の回路図を更新:
- Diagram4（反転昇降圧U4）の作業進行中
- LM2596S-ADJシンボルを正しいピン設定で追加
- 入力コンデンサC9（100µF）、C10（100nF）を正しい値で配置
- インダクタL3（100µH）、ダイオードD3（SS34）を追加
- 出力コンデンサC11（470µF 25V）を追加
- フィードバックネットワークR5（10k）、R6（1k）、C33（22nF）を追加
- ONピンをIC GNDに接続（ブートストラップトポロジ用）

リニアレギュレーション段の回路図を更新:
- コンポーネントシンボルと配線の改善
- 各レギュレータの入出力コンデンサ配置の明確化

次のステップ:
- TABピンを-13.5V OUT rail（IC GND）に接続
- すべての接続がDiagram4ドキュメントと一致することを確認
- PCBレイアウトでの配置検討

🤖 Generated with [Claude Code](https://claude.com/claude-code)

Co-Authored-By: Claude Sonnet 4.5 <noreply@anthropic.com>
Parts:
- renumbered UU1 to U1
Changed lines of the file:
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@@
 		(dnp no)
 		(fields_autoplaced yes)
-		(property "Reference" "UU1"
+		(property "Reference" "U1"
 			(at 152.4 30.48 0)
 			(effects
@@
 			(project ""
 				(path "/c5ce32ac-bd6d-413c-bfb5-5e9e2f8848d1/89c28db7-f9d9-4adf-b951-b9bb069eac97"
-					(reference "UU1")
+					(reference "U1")
 					(unit 1)
 				)
