File: usb-pd-input.kicad_sch (KiCad schematic)
At the start: 8 parts, among them J1 USB-C, U1 CH224D

Commit message: wip
Connections:
- net at J1.A5 (CC1), R13.2, U1.10 (CC1): no longer R12.2
- net at J1.B5 (CC2), U1.11 (CC2): now also R12.2
Changed lines of the file:
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@@
-	)
-	(junction
-		(at 86.36 57.15)
-		(diameter 0)
-		(color 0 0 0 0)
 	)
 	(junction
@@
 	)
 	(junction
+		(at 86.36 54.61)
+		(diameter 0)
+		(color 0 0 0 0)
+	)
+	(junction
 		(at 69.85 96.52)
 		(diameter 0)
@@
 	(wire
 		(pts
+			(xy 86.36 54.61) (xy 86.36 63.5)
+		)
+		(stroke
+			(width 0)
+			(type default)
+		)
+	)
+	(wire
+		(pts
 			(xy 69.85 49.53) (xy 69.85 62.23)
 		)
@@
 	(wire
 		(pts
-			(xy 77.47 57.15) (xy 86.36 57.15)
-		)
-		(stroke
-			(width 0)
-			(type default)
-		)
-	)
-	(wire
-		(pts
 			(xy 168.91 96.52) (xy 163.83 96.52)
 		)
@@
 	(wire
 		(pts
-			(xy 86.36 57.15) (xy 86.36 63.5)
-		)
-		(stroke
-			(width 0)
-			(type default)
-		)
-	)
-	(wire
-		(pts
 			(xy 134.62 96.52) (xy 163.83 96.52)
 		)
@@
 	(wire
 		(pts
-			(xy 128.27 54.61) (xy 66.04 54.61)
+			(xy 128.27 54.61) (xy 86.36 54.61)
 		)
 		(stroke
@@
 	(wire
 		(pts
-			(xy 86.36 57.15) (xy 132.08 57.15)
+			(xy 77.47 57.15) (xy 132.08 57.15)
 		)
 		(stroke
@@
 		)
 		(stroke
+			(width 0)
+			(type default)
+		)
+	)
+	(wire
+		(pts
+			(xy 86.36 54.61) (xy 66.04 54.61)
+		)
+		(stroke

Commit message: === before edit sch ===
Connections:
- net GND: now also J1.7 (EH)
Other:
- moved on the sheet: C1, C2
