File: usb-pd-input.kicad_sch (KiCad schematic)
At the start: 23 parts, among them J1 USB-C, J2 Pogo pads, J3 Pogo pads (debug), Q1 -30V -4A, U1 STUSB4500QTR

Commit message: feat(usb-pd): apply JLCPCB pre-production LCSC part swaps for v3
- C4/C22/C23 (470µF 16V): C46550400 → C970706 (DMBJ RVT1C471M0810, D8×L10.2mm)
- C2/C6/C8/C10/C17/C18/C19/C35 (100nF 50V X7R 0805): C49678 → C1711 (Samsung CL21B104KBCNNNC)
- R12 (56k 0603): align BOM C23168 → C23206 (Uniroyal) to match schematic

Updated LCSC Part properties in dc-dc-conversion, linear-regulation, and usb-pd-input schematics.
Parts:
- C2, C35: LCSC Part C28233 -> C1711
Changed lines of the file:
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@@
 			)
 		)
-		(property "LCSC Part" "C28233"
+		(property "LCSC Part" "C1711"
 			(at 203.2 121.92 0)
 			(hide yes)
@@
 			)
 		)
-		(property "LCSC Part" "C28233"
+		(property "LCSC Part" "C1711"
 			(at 229.87 21.59 0)
 			(hide yes)
