File: experiments/ai-circuit-design/circuit-synth-spike/generated_linear_regulation/neg_12v_stage.kicad_sch (KiCad schematic)
At the start: 9 parts

Commit message: fix(experiments): address deep-review findings (SPICE model, LED polarity, skill perms)
Codex review (P2) fixes on the A–D trial artifacts:
- SPICE value-sizing deck: the loop-closed check pinned FB to Vref via an ideal
  source, which floated VOUT (KCL forced VOUT==FB≈1.23V). Replaced with a
  high-gain error-amp behavioral source driving the real divider, so .op now
  genuinely solves VOUT=Vref*(1+Rtop/Rbot). Same fix in the sweep deck; FINDINGS
  method note updated.
- circuit-synth spike: Device:LED pin1=cathode/pin2=anode, but the helper wired
  the positive rail to pin1 → reverse-biased +12V/+5V indicator LEDs. Added a
  rail-aware `negative` flag; positive stages now anode→rail, negative stage
  anode→GND. Regenerated the .kicad_sch/.net/.json output to match.
- pd-schematic-review skill: added `Bash(mkdir -p __inbox*)` to allowed-tools so
  the netlist-export step doesn't block on a fresh clone (__inbox is gitignored).

Co-Authored-By: Claude Opus 4.8 (1M context) <noreply@anthropic.com>
Parts:
- C10, C11, C12, C9, D3, F3, LED3, R3, U8: hierarchy_path /dee5fd78-2d54-41fe-ba07-6c5be7c122e4/e095d0ab-1423-4974-8e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 -> /fde22f73-ec7e-4a79-83c1-d101e011a27c/55f139b1-41df-4a00-af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; root_uuid dee5fd78-2d54-41fe-ba07-6c5be7c122e4 -> fde22f73-ec7e-4a79-83c1-d101e011a27c
Changed lines of the file:
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@@
 			)
 		)
-		(property "hierarchy_path" "/dee5fd78-2d54-41fe-ba07-6c5be7c122e4/e095d0ab-1423-4974-8ee4-13d6d2b23241"
+		(property "hierarchy_path" "/fde22f73-ec7e-4a79-83c1-d101e011a27c/55f139b1-41df-4a00-af9f-303ea778c188"
 			(at 40.64 35.5599 0)
 			(effects
@@
 			)
 		)
-		(property "root_uuid" "dee5fd78-2d54-41fe-ba07-6c5be7c122e4"
+		(property "root_uuid" "fde22f73-ec7e-4a79-83c1-d101e011a27c"
 			(at 40.64 35.5599 0)
 			(effects
@@
 		(instances
 			(project ""
-				(path "/dee5fd78-2d54-41fe-ba07-6c5be7c122e4/e095d0ab-1423-4974-8ee4-13d6d2b23241"
+				(path "/fde22f73-ec7e-4a79-83c1-d101e011a27c/55f139b1-41df-4a00-af9f-303ea778c188"
 					(reference "U8")
 					(unit 1)
@@
 			)
 		)
-		(property "hierarchy_path" "/dee5fd78-2d54-41fe-ba07-6c5be7c122e4/e095d0ab-1423-4974-8ee4-13d6d2b23241"
+		(property "hierarchy_path" "/fde22f73-ec7e-4a79-83c1-d101e011a27c/55f139b1-41df-4a00-af9f-303ea778c188"
 			(at 187.96 38.0999 0)
 			(effects
@@
 			)
 		)
-		(property "root_uuid" "dee5fd78-2d54-41fe-ba07-6c5be7c122e4"
+		(property "root_uuid" "fde22f73-ec7e-4a79-83c1-d101e011a27c"
 			(at 187.96 38.0999 0)
 			(effects
@@
 		(instances
 			(project ""
-				(path "/dee5fd78-2d54-41fe-ba07-6c5be7c122e4/e095d0ab-1423-4974-8ee4-13d6d2b23241"
+				(path "/fde22f73-ec7e-4a79-83c1-d101e011a27c/55f139b1-41df-4a00-af9f-303ea778c188"
 					(reference "C9")
 					(unit 1)
@@
 			)
 		)
-		(property "hierarchy_path" "/dee5fd78-2d54-41fe-ba07-6c5be7c122e4/e095d0ab-1423-4974-8ee4-13d6d2b23241"
+		(property "hierarchy_path" "/fde22f73-ec7e-4a79-83c1-d101e011a27c/55f139b1-41df-4a00-af9f-303ea778c188"
 			(at 213.36 38.0999 0)
 			(effects
@@
 			)
 		)
-		(property "root_uuid" "dee5fd78-2d54-41fe-ba07-6c5be7c122e4"
+		(property "root_uuid" "fde22f73-ec7e-4a79-83c1-d101e011a27c"
 			(at 213.36 38.0999 0)
 			(effects
@@
 		(instances
 			(project ""
-				(path "/dee5fd78-2d54-41fe-ba07-6c5be7c122e4/e095d0ab-1423-4974-8ee4-13d6d2b23241"
+				(path "/fde22f73-ec7e-4a79-83c1-d101e011a27c/55f139b1-41df-4a00-af9f-303ea778c188"
 					(reference "C10")
 					(unit 1)
@@
 			)
 		)
-		(property "hierarchy_path" "/dee5fd78-2d54-41fe-ba07-6c5be7c122e4/e095d0ab-1423-4974-8ee4-13d6d2b23241"
+		(property "hierarchy_path" "/fde22f73-ec7e-4a79-83c1-d101e011a27c/55f139b1-41df-4a00-af9f-303ea778c188"
 			(at 238.76 38.0999 0)
 			(effects
@@
 			)
 		)
-		(property "root_uuid" "dee5fd78-2d54-41fe-ba07-6c5be7c122e4"
+		(property "root_uuid" "fde22f73-ec7e-4a79-83c1-d101e011a27c"
 			(at 238.76 38.0999 0)
 			(effects
@@
 		(instances
 			(project ""
-				(path "/dee5fd78-2d54-41fe-ba07-6c5be7c122e4/e095d0ab-1423-4974-8ee4-13d6d2b23241"
+				(path "/fde22f73-ec7e-4a79-83c1-d101e011a27c/55f139b1-41df-4a00-af9f-303ea778c188"
 					(reference "C11")
 					(unit 1)
@@
 			)
 		)
-		(property "hierarchy_path" "/dee5fd78-2d54-41fe-ba07-6c5be7c122e4/e095d0ab-1423-4974-8ee4-13d6d2b23241"
+		(property "hierarchy_path" "/fde22f73-ec7e-4a79-83c1-d101e011a27c/55f139b1-41df-4a00-af9f-303ea778c188"
 			(at 264.16 38.0999 0)
 			(effects
@@
 			)
 		)
-		(property "root_uuid" "dee5fd78-2d54-41fe-ba07-6c5be7c122e4"
+		(property "root_uuid" "fde22f73-ec7e-4a79-83c1-d101e011a27c"
 			(at 264.16 38.0999 0)
 			(effects
@@
 		(instances
 			(project ""
-				(path "/dee5fd78-2d54-41fe-ba07-6c5be7c122e4/e095d0ab-1423-4974-8ee4-13d6d2b23241"
+				(path "/fde22f73-ec7e-4a79-83c1-d101e011a27c/55f139b1-41df-4a00-af9f-303ea778c188"
 					(reference "C12")
 					(unit 1)
@@
 			)
 		)
-		(property "hierarchy_path" "/dee5fd78-2d54-41fe-ba07-6c5be7c122e4/e095d0ab-1423-4974-8ee4-13d6d2b23241"
+		(property "hierarchy_path" "/fde22f73-ec7e-4a79-83c1-d101e011a27c/55f139b1-41df-4a00-af9f-303ea778c188"
 			(at 73.66 40.6399 0)
 			(effects
@@
 			)
 		)
-		(property "root_uuid" "dee5fd78-2d54-41fe-ba07-6c5be7c122e4"
+		(property "root_uuid" "fde22f73-ec7e-4a79-83c1-d101e011a27c"
 			(at 73.66 40.6399 0)
 			(effects
@@
 		(instances
 			(project ""
-				(path "/dee5fd78-2d54-41fe-ba07-6c5be7c122e4/e095d0ab-1423-4974-8ee4-13d6d2b23241"
+				(path "/fde22f73-ec7e-4a79-83c1-d101e011a27c/55f139b1-41df-4a00-af9f-303ea778c188"
 					(reference "F3")
 					(unit 1)
@@
 			)
 		)
-		(property "hierarchy_path" "/dee5fd78-2d54-41fe-ba07-6c5be7c122e4/e095d0ab-1423-4974-8ee4-13d6d2b23241"
+		(property "hierarchy_path" "/fde22f73-ec7e-4a79-83c1-d101e011a27c/55f139b1-41df-4a00-af9f-303ea778c188"
 			(at 160.02 30.4799 0)
 			(effects
@@
 			)
 		)
-		(property "root_uuid" "dee5fd78-2d54-41fe-ba07-6c5be7c122e4"
+		(property "root_uuid" "fde22f73-ec7e-4a79-83c1-d101e011a27c"
 			(at 160.02 30.4799 0)
 			(effects
@@
 		(instances
 			(project ""
-				(path "/dee5fd78-2d54-41fe-ba07-6c5be7c122e4/e095d0ab-1423-4974-8ee4-13d6d2b23241"
+				(path "/fde22f73-ec7e-4a79-83c1-d101e011a27c/55f139b1-41df-4a00-af9f-303ea778c188"
 					(reference "D3")
 					(unit 1)
@@
 			)
 		)
-		(property "hierarchy_path" "/dee5fd78-2d54-41fe-ba07-6c5be7c122e4/e095d0ab-1423-4974-8ee4-13d6d2b23241"
+		(property "hierarchy_path" "/fde22f73-ec7e-4a79-83c1-d101e011a27c/55f139b1-41df-4a00-af9f-303ea778c188"
 			(at 96.52 40.6399 0)
 			(effects
@@
 			)
 		)
-		(property "root_uuid" "dee5fd78-2d54-41fe-ba07-6c5be7c122e4"
+		(property "root_uuid" "fde22f73-ec7e-4a79-83c1-d101e011a27c"
 			(at 96.52 40.6399 0)
 			(effects
@@
 		(instances
 			(project ""
-				(path "/dee5fd78-2d54-41fe-ba07-6c5be7c122e4/e095d0ab-1423-4974-8ee4-13d6d2b23241"
+				(path "/fde22f73-ec7e-4a79-83c1-d101e011a27c/55f139b1-41df-4a00-af9f-303ea778c188"
 					(reference "R3")
 					(unit 1)
@@
 			)
 		)
-		(property "hierarchy_path" "/dee5fd78-2d54-41fe-ba07-6c5be7c122e4/e095d0ab-1423-4974-8ee4-13d6d2b23241"
+		(property "hierarchy_path" "/fde22f73-ec7e-4a79-83c1-d101e011a27c/55f139b1-41df-4a00-af9f-303ea778c188"
 			(at 127 30.4799 0)
 			(effects
@@
 			)
 		)
-		(property "root_uuid" "dee5fd78-2d54-41fe-ba07-6c5be7c122e4"
+		(property "root_uuid" "fde22f73-ec7e-4a79-83c1-d101e011a27c"
 			(at 127 30.4799 0)
 			(effects
@@
 		(instances
 			(project ""
-				(path "/dee5fd78-2d54-41fe-ba07-6c5be7c122e4/e095d0ab-1423-4974-8ee4-13d6d2b23241"
+				(path "/fde22f73-ec7e-4a79-83c1-d101e011a27c/55f139b1-41df-4a00-af9f-303ea778c188"
 					(reference "LED3")
 					(unit 1)
