File: boards/board-p/board-p.kicad_pcb (KiCad board)
At the start: 2 copper layers, 27 x 40 mm, 28 parts, among them J1 TYPE-C-31-M-17, J2 PogoPad_1x4_NVM_I2C, J3 PogoPad_1x8_Debug, Q1 AO3401A, U1 STUSB4500QTR

Commit message: fix(board-p): replace out-of-stock D5 TVS with Littelfuse SMAJ16A (C74561)
Vishay SMAJ16A-E3/61 (C968650) was out of stock at JLCPCB. Footprint pads and package updated; schematic routing unchanged.

Co-Authored-By: Claude Fable 5.1 <noreply@anthropic.com>
Parts:
- D5: value SMAJ16A-E3/61 -> SMAJ16A; footprint zudo-pd:SMA_Vishay_SMAJ16A_C968650 -> zudo-pd:SMA_Littelfuse_SMAJ16A_C74561
Changed lines of the file:
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@@
 		)
 	)
-	(footprint "zudo-pd:SMA_Vishay_SMAJ16A_C968650"
+	(footprint "zudo-pd:SMA_Littelfuse_SMAJ16A_C74561"
 		(layer "F.Cu")
 		(at 22.25 10.08)
@@
 			)
 		)
-		(property "Value" "SMAJ16A-E3/61"
+		(property "Value" "SMAJ16A"
 			(at 0 4 0)
 			(layer "F.Fab")
@@
 			)
 		)
-		(property "LCSC Part" "C968650"
+		(property "LCSC Part" "C74561"
 			(at 0 0 0)
 			(layer "F.Fab")
@@
 			)
 		)
-		(property "LCSC" "C968650"
+		(property "LCSC" "C74561"
 			(at 0 0 0)
 			(unlocked yes)
@@
 		)
 		(fp_line
-			(start -2.95 -1.65)
-			(end 2.95 -1.65)
+			(start -3.1 -1.65)
+			(end 3.1 -1.65)
 			(stroke
 				(width 0.05)
@@
 		)
 		(fp_line
-			(start -2.95 1.65)
-			(end -2.95 -1.65)
+			(start -3.1 1.65)
+			(end -3.1 -1.65)
 			(stroke
 				(width 0.05)
@@
 		)
 		(fp_line
-			(start 2.95 -1.65)
-			(end 2.95 1.65)
+			(start 3.1 -1.65)
+			(end 3.1 1.65)
 			(stroke
 				(width 0.05)
@@
 		)
 		(fp_line
-			(start 2.95 1.65)
-			(end -2.95 1.65)
+			(start 3.1 1.65)
+			(end -3.1 1.65)
 			(stroke
 				(width 0.05)
@@
 		(pad "1" smd rect
 			(at -1.8 0)
-			(size 1.8 1.8)
+			(size 2.1 1.8)
 			(layers "F.Cu" "F.Mask" "F.Paste")
 			(net "VBUS_IN")
@@
 		(pad "2" smd rect
 			(at 1.8 0)
-			(size 1.8 1.8)
+			(size 2.1 1.8)
 			(layers "F.Cu" "F.Mask" "F.Paste")
 			(net "GND")
 		)
 		(embedded_fonts no)
-		(model "${KIPRJMOD}/../../footprints/kicad/zudo-pd.3dshapes/SMA_Vishay_SMAJ16A_C968650.wrl"
+		(model "${KIPRJMOD}/../../footprints/kicad/zudo-pd.3dshapes/SMA_Littelfuse_SMAJ16A_C74561.wrl"
 			(offset
 				(xyz 0 0 0)
