File: boards/board-p/board-p.kicad_sch (KiCad schematic)
At the start: 25 parts, among them J1 TYPE-C-31-M-17, J2 PogoPad_1x4_NVM_I2C, J3 PogoPad_1x8_Debug, Q1 AO3401A, U1 STUSB4500QTR

Commit message: fix(board-p): replace out-of-stock D5 TVS with Littelfuse SMAJ16A (C74561)
Vishay SMAJ16A-E3/61 (C968650) was out of stock at JLCPCB. Footprint pads and package updated; schematic routing unchanged.

Co-Authored-By: Claude Fable 5.1 <noreply@anthropic.com>
Parts:
- D5: value SMAJ16A-E3/61 -> SMAJ16A; footprint zudo-pd:SMA_Vishay_SMAJ16A_C968650 -> zudo-pd:SMA_Littelfuse_SMAJ16A_C74561; symbol zudo-pd:SMAJ16A-E3/61 -> zudo-pd:SMAJ16A; LCSC C968650 -> C74561
Changed lines of the file:
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@@
 	)
 	(symbol
-		(lib_id "zudo-pd:SMAJ16A-E3/61")
+		(lib_id "zudo-pd:SMAJ16A")
 		(at 203.2 38.1 0)
 		(unit 1)
@@
 			)
 		)
-		(property "Value" "SMAJ16A-E3/61"
+		(property "Value" "SMAJ16A"
 			(at 203.2 43.18 0)
 			(effects
@@
 			)
 		)
-		(property "Footprint" "zudo-pd:SMA_Vishay_SMAJ16A_C968650"
+		(property "Footprint" "zudo-pd:SMA_Littelfuse_SMAJ16A_C74561"
 			(at 203.2 38.1 0)
 			(effects
@@
 			)
 		)
-		(property "LCSC" "C968650"
+		(property "LCSC" "C74561"
 			(at 203.2 45.72 0)
 			(effects
