File: manufacturing/releases/corner-support-review/board-p/source/board-p.kicad_pcb (KiCad board)
At the start: 2 copper layers, 27 x 40 mm, 28 parts, among them J1 TYPE-C-31-M-17, J2 PogoPad_1x4_NVM_I2C, J3 PogoPad_1x8_Debug, Q1 AO3401A, U1 STUSB4500QTR

Commit message: build: regenerate assembly preview, leg fit evidence and prototype package for D5 change
Assembly preview, PCB leg fit evidence and manufacturing release package updated for D5 TVS footprint change.

Co-Authored-By: Claude Fable 5.1 <noreply@anthropic.com>
Parts:
- D5: value SMAJ16A-E3/61 -> SMAJ16A; footprint zudo-pd:SMA_Vishay_SMAJ16A_C968650 -> zudo-pd:SMA_Littelfuse_SMAJ16A_C74561
Changed lines of the file:
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@@
 		)
 		(embedded_fonts no)
-		(model "${KIPRJMOD}/../../../../../footprints/kicad/zudo-pd.3dshapes/QFN-24_L4.0-W4.0-P0.50-BL-EP2.8.wrl"
+		(model "${KIPRJMOD}/../../../../footprints/kicad/zudo-pd.3dshapes/QFN-24_L4.0-W4.0-P0.50-BL-EP2.8.wrl"
 			(offset
 				(xyz 0 0 0)
@@
 		)
 	)
-	(footprint "zudo-pd:SMA_Vishay_SMAJ16A_C968650"
+	(footprint "zudo-pd:SMA_Littelfuse_SMAJ16A_C74561"
 		(layer "F.Cu")
 		(at 22.25 10.08)
@@
 			)
 		)
-		(property "Value" "SMAJ16A-E3/61"
+		(property "Value" "SMAJ16A"
 			(at 0 4 0)
 			(layer "F.Fab")
@@
 			)
 		)
-		(property "LCSC Part" "C968650"
+		(property "LCSC Part" "C74561"
 			(at 0 0 0)
 			(layer "F.Fab")
@@
 			)
 		)
-		(property "LCSC" "C968650"
+		(property "LCSC" "C74561"
 			(at 0 0 0)
 			(unlocked yes)
@@
 		)
 		(fp_line
-			(start -2.95 -1.65)
-			(end 2.95 -1.65)
+			(start -3.1 -1.65)
+			(end 3.1 -1.65)
 			(stroke
 				(width 0.05)
@@
 		)
 		(fp_line
-			(start -2.95 1.65)
-			(end -2.95 -1.65)
+			(start -3.1 1.65)
+			(end -3.1 -1.65)
 			(stroke
 				(width 0.05)
@@
 		)
 		(fp_line
-			(start 2.95 -1.65)
-			(end 2.95 1.65)
+			(start 3.1 -1.65)
+			(end 3.1 1.65)
 			(stroke
 				(width 0.05)
@@
 		)
 		(fp_line
-			(start 2.95 1.65)
-			(end -2.95 1.65)
+			(start 3.1 1.65)
+			(end -3.1 1.65)
 			(stroke
 				(width 0.05)
@@
 		(pad "1" smd rect
 			(at -1.8 0)
-			(size 1.8 1.8)
+			(size 2.1 1.8)
 			(layers "F.Cu" "F.Mask" "F.Paste")
 			(net "VBUS_IN")
@@
 		(pad "2" smd rect
 			(at 1.8 0)
-			(size 1.8 1.8)
+			(size 2.1 1.8)
 			(layers "F.Cu" "F.Mask" "F.Paste")
 			(net "GND")
 		)
 		(embedded_fonts no)
-		(model "${KIPRJMOD}/../../../../../footprints/kicad/zudo-pd.3dshapes/SMA_Vishay_SMAJ16A_C968650.wrl"
+		(model "${KIPRJMOD}/../../../../footprints/kicad/zudo-pd.3dshapes/SMA_Littelfuse_SMAJ16A_C74561.wrl"
 			(offset
 				(xyz 0 0 0)
@@
 		)
 		(embedded_fonts no)
-		(model "${KIPRJMOD}/../../../../../footprints/kicad/zudo-pd.3dshapes/C0603_L1.6-W0.8-H0.8.wrl"
+		(model "${KIPRJMOD}/../../../../footprints/kicad/zudo-pd.3dshapes/C0603_L1.6-W0.8-H0.8.wrl"
 			(offset
 				(xyz 0 0 0)
@@
 		)
 		(embedded_fonts no)
-		(model "${KIPRJMOD}/../../../../../footprints/kicad/zudo-pd.3dshapes/R0603.wrl"
+		(model "${KIPRJMOD}/../../../../footprints/kicad/zudo-pd.3dshapes/R0603.wrl"
 			(offset
 				(xyz 0 0 0)
@@
 		)
 		(embedded_fonts no)
-		(model "${KIPRJMOD}/../../../../../footprints/kicad/zudo-pd.3dshapes/R0603.wrl"
+		(model "${KIPRJMOD}/../../../../footprints/kicad/zudo-pd.3dshapes/R0603.wrl"
 			(offset
 				(xyz 0 0 0)
@@
 		)
 		(embedded_fonts no)
-		(model "${KIPRJMOD}/../../../../../footprints/kicad/zudo-pd.3dshapes/SOT-23-3P_L2.9-W1.3-H1.0-LS2.4-P0.95.wrl"
+		(model "${KIPRJMOD}/../../../../footprints/kicad/zudo-pd.3dshapes/SOT-23-3P_L2.9-W1.3-H1.0-LS2.4-P0.95.wrl"
 			(offset
 				(xyz 0 0 0)
@@
 		)
 		(embedded_fonts no)
-		(model "${KIPRJMOD}/../../../../../footprints/kicad/zudo-pd.3dshapes/C0603_L1.6-W0.8-H0.8.wrl"
+		(model "${KIPRJMOD}/../../../../footprints/kicad/zudo-pd.3dshapes/C0603_L1.6-W0.8-H0.8.wrl"
 			(offset
 				(xyz 0 0 0)
@@
 		)
 		(embedded_fonts no)
-		(model "${KIPRJMOD}/../../../../../footprints/kicad/zudo-pd.3dshapes/R0603.wrl"
+		(model "${KIPRJMOD}/../../../../footprints/kicad/zudo-pd.3dshapes/R0603.wrl"
 			(offset
 				(xyz 0 0 0)
@@
 		)
 		(embedded_fonts no)
-		(model "${KIPRJMOD}/../../../../../footprints/kicad/zudo-pd.3dshapes/R0603.wrl"
+		(model "${KIPRJMOD}/../../../../footprints/kicad/zudo-pd.3dshapes/R0603.wrl"
 			(offset
 				(xyz 0 0 0)
@@
 		)
 		(embedded_fonts no)
-		(model "${KIPRJMOD}/../../../../../footprints/kicad/zudo-pd.3dshapes/SOD-523_L1.2-W0.8-H0.7-LS1.6.wrl"
+		(model "${KIPRJMOD}/../../../../footprints/kicad/zudo-pd.3dshapes/SOD-523_L1.2-W0.8-H0.7-LS1.6.wrl"
 			(offset
 				(xyz 0 0 0)
@@
 		)
 		(embedded_fonts no)
-		(model "${KIPRJMOD}/../../../../../footprints/kicad/zudo-pd.3dshapes/USB-C-SMD_10P-P1.00-L6.8-W8.9.wrl"
+		(model "${KIPRJMOD}/../../../../footprints/kicad/zudo-pd.3dshapes/USB-C-SMD_10P-P1.00-L6.8-W8.9.wrl"
 			(offset
 				(xyz 0 -2.468 0)
@@
 		)
 		(embedded_fonts no)
-		(model "${KIPRJMOD}/../../../../../footprints/kicad/zudo-pd.3dshapes/R0603.wrl"
+		(model "${KIPRJMOD}/../../../../footprints/kicad/zudo-pd.3dshapes/R0603.wrl"
 			(offset
 				(xyz 0 0 0)
@@
 		)
 		(embedded_fonts no)
-		(model "${KIPRJMOD}/../../../../../footprints/kicad/zudo-pd.3dshapes/R0603.wrl"
+		(model "${KIPRJMOD}/../../../../footprints/kicad/zudo-pd.3dshapes/R0603.wrl"
 			(offset
 				(xyz 0 0 0)
@@
 		)
 		(embedded_fonts no)
-		(model "${KIPRJMOD}/../../../../../footprints/kicad/zudo-pd.3dshapes/R0603.wrl"
+		(model "${KIPRJMOD}/../../../../footprints/kicad/zudo-pd.3dshapes/R0603.wrl"
 			(offset
 				(xyz 0 0 0)
@@
 		)
 		(embedded_fonts no)
-		(model "${KIPRJMOD}/../../../../../footprints/kicad/zudo-pd.3dshapes/C0603_L1.6-W0.8-H0.8.wrl"
+		(model "${KIPRJMOD}/../../../../footprints/kicad/zudo-pd.3dshapes/C0603_L1.6-W0.8-H0.8.wrl"
 			(offset
 				(xyz 0 0 0)
@@
 		)
 		(embedded_fonts no)
-		(model "${KIPRJMOD}/../../../../../footprints/kicad/zudo-pd.3dshapes/HDR-TH_6P-P2.54-M-LI-1X6P.wrl"
+		(model "${KIPRJMOD}/../../../../footprints/kicad/zudo-pd.3dshapes/HDR-TH_6P-P2.54-M-LI-1X6P.wrl"
 			(offset
 				(xyz 0 0 0)
@@
 		)
 		(embedded_fonts no)
-		(model "${KIPRJMOD}/../../../../../footprints/kicad/zudo-pd.3dshapes/R0603.wrl"
+		(model "${KIPRJMOD}/../../../../footprints/kicad/zudo-pd.3dshapes/R0603.wrl"
 			(offset
 				(xyz 0 0 0)
@@
 		)
 		(embedded_fonts no)
-		(model "${KIPRJMOD}/../../../../../footprints/kicad/zudo-pd.3dshapes/C0603_L1.6-W0.8-H0.8.wrl"
+		(model "${KIPRJMOD}/../../../../footprints/kicad/zudo-pd.3dshapes/C0603_L1.6-W0.8-H0.8.wrl"
 			(offset
 				(xyz 0 0 0)
@@
 		)
 		(embedded_fonts no)
-		(model "${KIPRJMOD}/../../../../../footprints/kicad/zudo-pd.3dshapes/R0603.wrl"
+		(model "${KIPRJMOD}/../../../../footprints/kicad/zudo-pd.3dshapes/R0603.wrl"
 			(offset
 				(xyz 0 0 0)
@@
 		)
 		(embedded_fonts no)
-		(model "${KIPRJMOD}/../../../../../footprints/kicad/zudo-pd.3dshapes/R0805_L2.0-W1.3-H0.6.wrl"
+		(model "${KIPRJMOD}/../../../../footprints/kicad/zudo-pd.3dshapes/R0805_L2.0-W1.3-H0.6.wrl"
 			(offset
 				(xyz 0 0 0)
@@
 		)
 		(embedded_fonts no)
-		(model "${KIPRJMOD}/../../../../../footprints/kicad/zudo-pd.3dshapes/SOD-523_L1.2-W0.8-H0.7-LS1.6.wrl"
+		(model "${KIPRJMOD}/../../../../footprints/kicad/zudo-pd.3dshapes/SOD-523_L1.2-W0.8-H0.7-LS1.6.wrl"
 			(offset
 				(xyz 0 0 0)
@@
 		)
 		(embedded_fonts no)
-		(model "${KIPRJMOD}/../../../../../footprints/kicad/zudo-pd.3dshapes/R0603.wrl"
+		(model "${KIPRJMOD}/../../../../footprints/kicad/zudo-pd.3dshapes/R0603.wrl"
 			(offset
 				(xyz 0 0 0)
@@
 		)
 		(embedded_fonts no)
-		(model "${KIPRJMOD}/../../../../../footprints/kicad/zudo-pd.3dshapes/C1206_L3.2-W1.6-H1.3.wrl"
+		(model "${KIPRJMOD}/../../../../footprints/kicad/zudo-pd.3dshapes/C1206_L3.2-W1.6-H1.3.wrl"
 			(offset
 				(xyz 0 0 0)
