File: boards/board-b/board-b.kicad_sch (KiCad schematic)
At the start: 76 parts, among them J10 DW254P-2X8-L0, J11 DW254P-2X8-L0, J5 PM254V-11-06-H85, J6 WJ500V-5.08-2P, J7 WJ500V-5.08-2P, P1 ATT/PDOK pads, U2 AP63201WU-7, U3 LM2596S-ADJ, U4 LM2596S-ADJ, U6 LT1963AEQ#PBF, U7 LT1963AEQ#PBF, U8 LT3015EQ-12#PBF

Commit message: fix(board-b): replace out-of-stock LDOs, add U8 ADJ divider, correct LED2 polarity
Replace U6/U7 LT1963AEQ#PBF (C107286) with LT1963AEQ#TRPBF (C459702);
U8 fixed LT3015EQ-12#PBF (C666307) with adjustable LT3015EQ#PBF (C666306)
and new R26/R27/R28 divider (nominal −12.054 V). Also: LED2 (C2289) symbol
pin numbering corrected to pin 1 = cathode per LCSC library and footprint
turned 180° with copper unchanged (JLCPCB preview showed it reversed);
front/back silkscreen tidied; P1 label rule in verify-compact-mechanics.py relaxed
to nearest-own-contact.

Co-Authored-By: Claude Fable 5.1 <noreply@anthropic.com>
Parts:
- added R26: 8200R 0.1%, zudo-pd:R0603, symbol zudo-pd:RT0603BRD078K2L
- added R27: 680R 0.1%, zudo-pd:R0603, symbol zudo-pd:RT0603BRD07680RL
- added R28: 1000R 0.1%, zudo-pd:R0603, symbol zudo-pd:RT0603BRD071KL
- U6, U7: value LT1963AEQ#PBF -> LT1963AEQ#TRPBF; symbol zudo-pd:LT1963AEQ#PBF -> zudo-pd:LT1963AEQ#TRPBF; LCSC C107286 -> C459702
- U8: value LT3015EQ-12#PBF -> LT3015EQ#PBF; symbol zudo-pd:LT3015EQ-12#PBF -> zudo-pd:LT3015EQ#PBF; LCSC C666307 -> C666306
Connections:
- net GND: now also LED2.1 (A), R28.2; no longer LED2.2 (K)
- net Net-(R7-LED2): now also LED2.2 (K); no longer LED2.1 (A)
- net Net-(U8-OUT): now also R26.1; no longer U8.4 (SENSE/ADJ)
- new net U8 ADJ: R27.2, R28.1, U8.4 (SENSE/ADJ)
- new net U8 FB upper series: R26.2, R27.1
Changed lines of the file:
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@@
 	)
 	(symbol
-		(lib_id "zudo-pd:LT1963AEQ#PBF")
+		(lib_id "zudo-pd:LT1963AEQ#TRPBF")
 		(at 76.2 101.6 0)
 		(unit 1)
@@
 			)
 		)
-		(property "Value" "LT1963AEQ#PBF"
+		(property "Value" "LT1963AEQ#TRPBF"
 			(at 76.2 125.73 0)
 			(effects
@@
 			)
 		)
-		(property "LCSC" "C107286"
+		(property "LCSC" "C459702"
 			(at 76.2 109.22 0)
 			(effects
@@
 	)
 	(symbol
-		(lib_id "zudo-pd:LT1963AEQ#PBF")
+		(lib_id "zudo-pd:LT1963AEQ#TRPBF")
 		(at 165.1 101.6 0)
 		(unit 1)
@@
 			)
 		)
-		(property "Value" "LT1963AEQ#PBF"
+		(property "Value" "LT1963AEQ#TRPBF"
 			(at 165.1 125.73 0)
 			(effects
@@
 			)
 		)
-		(property "LCSC" "C107286"
+		(property "LCSC" "C459702"
 			(at 165.1 109.22 0)
 			(effects
@@
 	)
 	(symbol
-		(lib_id "zudo-pd:LT3015EQ-12#PBF")
+		(lib_id "zudo-pd:LT3015EQ#PBF")
 		(at 254 101.6 0)
 		(unit 1)
@@
 			)
 		)
-		(property "Value" "LT3015EQ-12#PBF"
+		(property "Value" "LT3015EQ#PBF"
 			(at 254 109.22 0)
 			(effects
@@
 			)
 		)
-		(property "LCSC" "C666307"
+		(property "LCSC" "C666306"
 			(at 254 109.22 0)
 			(effects
@@
 	)
 	(symbol
+		(lib_id "zudo-pd:RT0603BRD078K2L")
+		(at 609.6 482.6 0)
+		(unit 1)
+		(exclude_from_sim no)
+		(in_bom yes)
+		(on_board yes)
+		(dnp no)
+		(property "Reference" "R26"
+			(at 609.6 477.52 0)
+			(effects
+				(font (size 1.27 1.27))
+			)
+		)
+		(property "Value" "8200R 0.1%"
+			(at 609.6 487.68 0)
+			(effects
+				(font (size 1.27 1.27))
+			)
+		)
+		(property "Footprint" "zudo-pd:R0603"
+			(at 609.6 482.6 0)
+			(effects
+				(font (size 1.27 1.27))
+				(hide yes)
+			)
+		)
+		(property "Datasheet" ""
+			(at 609.6 482.6 0)
+			(effects
+				(font (size 1.27 1.27))
+				(hide yes)
+			)
+		)
+		(property "LCSC" "C861589"
+			(at 609.6 490.22 0)
+			(effects
+				(font (size 1.27 1.27))
+				(hide yes)
+			)
+		)
+		(pin "2"
+		)
+		(pin "1"
+		)
+		(instances
+			(project "board-b"
+				(path "/3d627066-684f-577a-80b2-2a76742d5147"
+					(reference "R26")
+					(unit 1)
+				)
+			)
+		)
+	)
+	(symbol
+		(lib_id "zudo-pd:RT0603BRD07680RL")
+		(at 698.5 482.6 0)
+		(unit 1)
+		(exclude_from_sim no)
+		(in_bom yes)
+		(on_board yes)
+		(dnp no)
+		(property "Reference" "R27"
+			(at 698.5 477.52 0)
+			(effects
+				(font (size 1.27 1.27))
+			)
+		)
+		(property "Value" "680R 0.1%"
+			(at 698.5 487.68 0)
+			(effects
+				(font (size 1.27 1.27))
+			)
+		)
+		(property "Footprint" "zudo-pd:R0603"
+			(at 698.5 482.6 0)
+			(effects
+				(font (size 1.27 1.27))
+				(hide yes)
+			)
+		)
+		(property "Datasheet" ""
+			(at 698.5 482.6 0)
+			(effects
+				(font (size 1.27 1.27))
+				(hide yes)
+			)
+		)
+		(property "LCSC" "C861519"
+			(at 698.5 490.22 0)
+			(effects
+				(font (size 1.27 1.27))
+				(hide yes)
+			)
+		)
+		(pin "2"
+		)
+		(pin "1"
+		)
+		(instances
+			(project "board-b"
+				(path "/3d627066-684f-577a-80b2-2a76742d5147"
+					(reference "R27")
+					(unit 1)
+				)
+			)
+		)
+	)
+	(symbol
+		(lib_id "zudo-pd:RT0603BRD071KL")
+		(at 787.4 482.6 0)
+		(unit 1)
+		(exclude_from_sim no)
+		(in_bom yes)
+		(on_board yes)
+		(dnp no)
+		(property "Reference" "R28"
+			(at 787.4 477.52 0)
+			(effects
+				(font (size 1.27 1.27))
+			)
+		)
+		(property "Value" "1000R 0.1%"
+			(at 787.4 487.68 0)
+			(effects
+				(font (size 1.27 1.27))
+			)
+		)
+		(property "Footprint" "zudo-pd:R0603"
+			(at 787.4 482.6 0)
+			(effects
+				(font (size 1.27 1.27))
+				(hide yes)
+			)
+		)
+		(property "Datasheet" ""
+			(at 787.4 482.6 0)
+			(effects
+				(font (size 1.27 1.27))
+				(hide yes)
+			)
+		)
+		(property "LCSC" "C110776"
+			(at 787.4 490.22 0)
+			(effects
+				(font (size 1.27 1.27))
+				(hide yes)
+			)
+		)
+		(pin "2"
+		)
+		(pin "1"
+		)
+		(instances
+			(project "board-b"
+				(path "/3d627066-684f-577a-80b2-2a76742d5147"
+					(reference "R28")
+					(unit 1)
+				)
+			)
+		)
+	)
+	(symbol
 		(lib_id "zudo-pd:GRM32ER71H106KA12L")
 		(at 76.2 482.6 0)
@@
 	(global_label "GND"
 		(shape passive)
+		(at 792.48 482.6 0)
+		(effects
+			(font (size 1.27 1.27))
+			(justify left)
+		)
+	)
+	(global_label "GND"
+		(shape passive)
 		(at 613.41 431.8 0)
 		(effects
@@
 	(global_label "GND"
 		(shape passive)
-		(at 604.52 304.8 180)
+		(at 614.68 304.8 0)
 		(effects
 			(font (size 1.27 1.27))
-			(justify right)
+			(justify left)
 		)
 	)
@@
 	(global_label "Net-(U8-OUT)"
 		(shape passive)
-		(at 237.49 101.6 180)
+		(at 604.52 482.6 180)
 		(effects
 			(font (size 1.27 1.27))
@@
 		)
 	)
+	(global_label "U8 FB upper series"
+		(shape passive)
+		(at 614.68 482.6 0)
+		(effects
+			(font (size 1.27 1.27))
+			(justify left)
+		)
+	)
+	(global_label "U8 FB upper series"
+		(shape passive)
+		(at 693.42 482.6 180)
+		(effects
+			(font (size 1.27 1.27))
+			(justify right)
+		)
+	)
+	(global_label "U8 ADJ"
+		(shape passive)
+		(at 703.58 482.6 0)
+		(effects
+			(font (size 1.27 1.27))
+			(justify left)
+		)
+	)
+	(global_label "U8 ADJ"
+		(shape passive)
+		(at 782.32 482.6 180)
+		(effects
+			(font (size 1.27 1.27))
+			(justify right)
+		)
+	)
+	(global_label "U8 ADJ"
+		(shape passive)
+		(at 237.49 101.6 180)
+		(effects
+			(font (size 1.27 1.27))
+			(justify right)
+		)
+	)
 	(global_label "+12V rail"
 		(shape passive)
@@
 	(global_label "Net-(R7-LED2)"
 		(shape passive)
-		(at 614.68 304.8 0)
+		(at 604.52 304.8 180)
 		(effects
 			(font (size 1.27 1.27))
-			(justify left)
+			(justify right)
 		)
 	)
